Commit message: gait algorithm improvement

File: pigot_description/urdf/pigot_model.xacro (robot description, xacro)
@@ -3,7 +3,4 @@
   <xacro:property name="motor_torque" value="300"/>
   <xacro:property name="motor_vec" value="12.56"/>
-  <xacro:property name="link_1_mass" value="1"/>
-  <xacro:property name="link_2_mass" value="1"/>
-  <xacro:property name="link_3_mass" value="1"/>
   <xacro:property name="motor_damp" value="0.1"/>
   <xacro:property name="motor_fric" value="0"/>
@@ -15,12 +12,12 @@
         rpy="0 0 0" />
       <mass
-        value="10" />
-      <inertia
-        ixx="0.06666"
+        value="5" />
+      <inertia
+        ixx="0.0333"
         ixy="0"
         ixz="0"
-        iyy="0.06666"
+        iyy="0.0333"
         iyz="0"
-        izz="0.06666" />
+        izz="0.0333" />
     </inertial>
     <visual>
@@ -56,4 +53,13 @@
     <child
       link="box_link" />
+  </joint>
+  <link name="dummy">
+    </link>
+  <joint name="dummy_joint" type="fixed">
+    <origin
+      xyz="0 0 0.75"
+      rpy="0 0 0" />
+    <parent link="dummy"/>
+    <child link="body_link"/>
   </joint>
   <link

Commit message: arm simulation

File: pigot_description/urdf/pigot_model.xacro (robot description, xacro)
@@ -1,837 +1,6 @@
 <?xml version="1.0" ?>
 <robot name="pigot" xmlns:xacro="http://www.ros.org/wiki/xacro">
-  <xacro:property name="motor_torque" value="300"/>
-  <xacro:property name="motor_vec" value="12.56"/>
-  <xacro:property name="motor_damp" value="0.1"/>
-  <xacro:property name="motor_fric" value="0"/>
-  <link
-    name="box_link">
-    <inertial>
-      <origin
-        xyz="0 0 0"
-        rpy="0 0 0" />
-      <mass
-        value="5" />
-      <inertia
-        ixx="0.0333"
-        ixy="0"
-        ixz="0"
-        iyy="0.0333"
-        iyz="0"
-        izz="0.0333" />
-    </inertial>
-    <visual>
-      <origin
-        xyz="0 0 0"
-        rpy="0 0 0" />
-      <geometry>
-        <box size="0.2 0.2 0.2"/>
-      </geometry>
-      <material
-        name="">
-        <color
-          rgba="1 1 1 1" />
-      </material>
-    </visual>
-    <collision>
-      <origin
-        xyz="0 0 0"
-        rpy="0 0 0" />
-      <geometry>
-        <box size="0.2 0.2 0.2"/>
-      </geometry>
-    </collision>
-  </link>
-  <joint
-    name="body_link"
-    type="fixed">
-    <origin
-      xyz="0 -0.3 0.2"
-      rpy="0 0 0" />
-    <parent
-      link="body_link" />
-    <child
-      link="box_link" />
-  </joint>
-  <link name="dummy">
-    </link>
-  <joint name="dummy_joint" type="fixed">
-    <origin
-      xyz="0 0 0.75"
-      rpy="0 0 0" />
-    <parent link="dummy"/>
-    <child link="body_link"/>
-  </joint>
-  <link
-    name="body_link">
-    <inertial>
-      <origin
-        xyz="4.7665E-11 -9.774E-11 0"
-        rpy="0 0 0" />
-      <mass
-        value="25.117" />
-      <inertia
-        ixx="1.9268"
-        ixy="2.1744E-07"
-        ixz="6.0623E-11"
-        iyy="0.39868"
-        iyz="-7.9898E-07"
-        izz="2.1621" />
-    </inertial>
-    <visual>
-      <origin
-        xyz="0 0 0"
-        rpy="0 0 0" />
-      <geometry>
-        <mesh
-          filename="package://pigot_stl_model/meshes/body_link.STL" />
-      </geometry>
-      <material
-        name="">
-        <color
-          rgba="1 1 1 1" />
-      </material>
-    </visual>
-    <collision>
-      <origin
-        xyz="0 0 0"
-        rpy="0 0 0" />
-      <geometry>
-        <mesh
-          filename="package://pigot_stl_model/meshes/body_link.STL" />
-      </geometry>
-    </collision>
-  </link>
-  <link
-    name="lf_link_1">
-    <inertial>
-      <origin
-        xyz="-0.050197 1.6579E-09 0.025721"
-        rpy="0 0 0" />
-      <mass
-        value="3.2973" />
-      <inertia
-        ixx="0.0075672"
-        ixy="5.1432E-09"
-        ixz="-3.4681E-09"
-        iyy="0.0078331"
-        iyz="2.7873E-09"
-        izz="0.0045551" />
-    </inertial>
-    <visual>
-      <origin
-        xyz="0 0 0"
-        rpy="0 0 0" />
-      <geometry>
-        <mesh
-          filename="package://pigot_stl_model/meshes/lf_link_1.STL" />
-      </geometry>
-      <material
-        name="">
-        <color
-          rgba="1 0.72157 0.32941 1" />
-      </material>
-    </visual>
-    <collision>
-      <origin
-        xyz="0 0 0"
-        rpy="0 0 0" />
-      <geometry>
-        <mesh
-          filename="package://pigot_stl_model/meshes/lf_link_1.STL" />
-      </geometry>
-    </collision>
-  </link>
-  <joint
-    name="lf_rot_1"
-    type="revolute">
-    <origin
-      xyz="0.2 -0.3498 0"
-      rpy="1.5708 0 1.5708" />
-    <parent
-      link="body_link" />
-    <child
-      link="lf_link_1" />
-    <axis
-      xyz="-1 0 0" />
-    <limit
-      lower="-1.57"
-      upper="1.57"
-      effort="${motor_torque}"
-      velocity="${motor_vec}" />
-    <dynamics
-      damping="${motor_damp}"
-      friction="${motor_fric}" />
-  </joint>
-  <link
-    name="lf_link_2">
-    <inertial>
-      <origin
-        xyz="-0.05 -0.1259 0"
-        rpy="0 0 0" />
-      <mass
-        value="9.0227" />
-      <inertia
-        ixx="0.13447"
-        ixy="2.7733E-17"
-        ixz="-4.1134E-18"
-        iyy="0.020174"
-        iyz="2.5177E-17"
-        izz="0.13014" />
-    </inertial>
-    <visual>
-      <origin
-        xyz="0 0 0"
-        rpy="0 0 0" />
-      <geometry>
-        <mesh
-          filename="package://pigot_stl_model/meshes/lf_link_2.STL" />
-      </geometry>
-      <material
-        name="">
-        <color
-          rgba="1 1 1 1" />
-      </material>
-    </visual>
-    <collision>
-      <origin
-        xyz="0 0 0"
-        rpy="0 0 0" />
-      <geometry>
-        <mesh
-          filename="package://pigot_stl_model/meshes/lf_link_2.STL" />
-      </geometry>
-    </collision>
-  </link>
-  <joint
-    name="lf_rot_2"
-    type="revolute">
-    <origin
-      xyz="-0.050197 0 0.1"
-      rpy="0 1.5708 0" />
-    <parent
-      link="lf_link_1" />
-    <child
-      link="lf_link_2" />
-    <axis
-      xyz="1 0 0" />
-    <limit
-      lower="-3.14"
-      upper="3.14"
-      effort="${motor_torque}"
-      velocity="${motor_vec}" />
-    <dynamics
-      damping="${motor_damp}"
-      friction="${motor_fric}" />
-  </joint>
-  <link
-    name="lf_link_3">
-    <inertial>
-      <origin
-        xyz="-0.0325 -0.1327 7.0855E-10"
-        rpy="0 0 0" />
-      <mass
-        value="2.9673" />
-      <inertia
-        ixx="0.041846"
-        ixy="1.8339E-10"
-        ixz="3.4138E-09"
-        iyy="0.0022039"
-        iyz="3.2982E-10"
-        izz="0.041328" />
-    </inertial>
-    <visual>
-      <origin
-        xyz="0 0 0"
-        rpy="0 0 0" />
-      <geometry>
-        <mesh
-          filename="package://pigot_stl_model/meshes/lf_link_3.STL" />
-      </geometry>
-      <material
-        name="">
-        <color
-          rgba="1 1 1 1" />
-      </material>
-    </visual>
-    <collision>
-      <origin
-        xyz="0 0 0"
-        rpy="0 0 0" />
-      <geometry>
-        <mesh
-          filename="package://pigot_stl_model/meshes/lf_link_3.STL" />
-      </geometry>
-    </collision>
-  </link>
-  <joint
-    name="lf_rot_3"
-    type="revolute">
-    <origin
-      xyz="-0.0175 -0.35 0"
-      rpy="0 0 0" />
-    <parent
-      link="lf_link_2" />
-    <child
-      link="lf_link_3" />
-    <axis
-      xyz="1 0 0" />
-    <limit
-      lower="-3.14"
-      upper="3.14"
-      effort="${motor_torque}"
-      velocity="${motor_vec}" />
-    <dynamics
-      damping="${motor_damp}"
-      friction="${motor_fric}" />
-  </joint>
-  <link
-    name="rf_link_1">
-    <inertial>
-      <origin
-        xyz="-0.050197 4.7329E-09 0.025721"
-        rpy="0 0 0" />
-      <mass
-        value="3.2973" />
-      <inertia
-        ixx="0.0075672"
-        ixy="6.0059E-09"
-        ixz="-3.3928E-09"
-        iyy="0.0078331"
-        iyz="2.6669E-09"
-        izz="0.0045551" />
-    </inertial>
-    <visual>
-      <origin
-        xyz="0 0 0"
-        rpy="0 0 0" />
-      <geometry>
-        <mesh
-          filename="package://pigot_stl_model/meshes/rf_link_1.STL" />
-      </geometry>
-      <material
-        name="">
-        <color
-          rgba="1 0.72157 0.32941 1" />
-      </material>
-    </visual>
-    <collision>
-      <origin
-        xyz="0 0 0"
-        rpy="0 0 0" />
-      <geometry>
-        <mesh
-          filename="package://pigot_stl_model/meshes/rf_link_1.STL" />
-      </geometry>
-    </collision>
-  </link>
-  <joint
-    name="rf_rot_1"
-    type="revolute">
-    <origin
-      xyz="-0.2 -0.3498 0"
-      rpy="-1.5708 0 1.5708" />
-    <parent
-      link="body_link" />
-    <child
-      link="rf_link_1" />
-    <axis
-      xyz="1 0 0" />
-    <limit
-      lower="-1.57"
-      upper="1.57"
-      effort="${motor_torque}"
-      velocity="${motor_vec}" />
-    <dynamics
-      damping="${motor_damp}"
-      friction="${motor_fric}" />
-  </joint>
-  <link
-    name="rf_link_2">
-    <inertial>
-      <origin
-        xyz="-0.05 -0.125901750874251 0"
-        rpy="0 0 0" />
-      <mass
-        value="9.02267120345913" />
-      <inertia
-        ixx="0.134474751410522"
-        ixy="-1.00856843872561E-18"
-        ixz="-3.2778892928792E-18"
-        iyy="0.0201741931777721"
-        iyz="-2.89770588449339E-18"
-        izz="0.130137705098105" />
-    </inertial>
-    <visual>
-      <origin
-        xyz="0 0 0"
-        rpy="0 0 0" />
-      <geometry>
-        <mesh
-          filename="package://pigot_stl_model/meshes/rf_link_2.STL" />
-      </geometry>
-      <material
-        name="">
-        <color
-          rgba="1 1 1 1" />
-      </material>
-    </visual>
-    <collision>
-      <origin
-        xyz="0 0 0"
-        rpy="0 0 0" />
-      <geometry>
-        <mesh
-          filename="package://pigot_stl_model/meshes/rf_link_2.STL" />
-      </geometry>
-    </collision>
-  </link>
-  <joint
-    name="rf_rot_2"
-    type="revolute">
-    <origin
-      xyz="-0.050197 0 0.1"
-      rpy="3.1416 1.5708 0" />
-    <parent
-      link="rf_link_1" />
-    <child
-      link="rf_link_2" />
-    <axis
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
File: pigot_description/urdf/pigot_trans.xacro (robot description, xacro)
@@ -1,123 +1,49 @@
 <?xml version="1.0" ?>
 <robot name="pigot" xmlns:xacro="http://www.ros.org/wiki/xacro">
-  <transmission name="lf_rot_1_trans">
-    <type>transmission_interface/SimpleTransmission</type>
-    <joint name="lf_rot_1">
-      <hardwareInterface>hardware_interface/EffortJointInterface</hardwareInterface>
-    </joint>
-    <actuator name="lf_rot_1_motor">
-      <hardwareInterface>hardware_interface/EffortJointInterface</hardwareInterface>
-      <mechanicalReduction>1</mechanicalReduction>
-    </actuator>
-  </transmission>
-  <transmission name="lf_rot_2_trans">
-    <type>transmission_interface/SimpleTransmission</type>
-    <joint name="lf_rot_2">
-      <hardwareInterface>hardware_interface/EffortJointInterface</hardwareInterface>
-    </joint>
-    <actuator name="lf_rot_2_motor">
-      <hardwareInterface>hardware_interface/EffortJointInterface</hardwareInterface>
-      <mechanicalReduction>1</mechanicalReduction>
-    </actuator>
-  </transmission>
-  <transmission name="lf_rot_3_trans">
-    <type>transmission_interface/SimpleTransmission</type>
-    <joint name="lf_rot_3">
-      <hardwareInterface>hardware_interface/EffortJointInterface</hardwareInterface>
-    </joint>
-    <actuator name="lf_rot_3_motor">
-      <hardwareInterface>hardware_interface/EffortJointInterface</hardwareInterface>
-      <mechanicalReduction>1</mechanicalReduction>
-    </actuator>
-  </transmission>
-  <transmission name="rf_rot_1_trans">
-    <type>transmission_interface/SimpleTransmission</type>
-    <joint name="rf_rot_1">
-      <hardwareInterface>hardware_interface/EffortJointInterface</hardwareInterface>
-    </joint>
-    <actuator name="rf_rot_1_motor">
-      <hardwareInterface>hardware_interface/EffortJointInterface</hardwareInterface>
-      <mechanicalReduction>1</mechanicalReduction>
-    </actuator>
-  </transmission>
-  <transmission name="rf_rot_2_trans">
-    <type>transmission_interface/SimpleTransmission</type>
-    <joint name="rf_rot_2">
-      <hardwareInterface>hardware_interface/EffortJointInterface</hardwareInterface>
-    </joint>
-    <actuator name="rf_rot_2_motor">
-      <hardwareInterface>hardware_interface/EffortJointInterface</hardwareInterface>
-      <mechanicalReduction>1</mechanicalReduction>
-    </actuator>
-  </transmission>
-  <transmission name="rf_rot_3_trans">
-    <type>transmission_interface/SimpleTransmission</type>
-    <joint name="rf_rot_3">
-      <hardwareInterface>hardware_interface/EffortJointInterface</hardwareInterface>
-    </joint>
-    <actuator name="rf_rot_3_motor">
-      <hardwareInterface>hardware_interface/EffortJointInterface</hardwareInterface>
-      <mechanicalReduction>1</mechanicalReduction>
-    </actuator>
-  </transmission>
-  <transmission name="lb_rot_1_trans">
-    <type>transmission_interface/SimpleTransmission</type>
-    <joint name="lb_rot_1">
-      <hardwareInterface>hardware_interface/EffortJointInterface</hardwareInterface>
-    </joint>
-    <actuator name="lb_rot_1_motor">
-      <hardwareInterface>hardware_interface/EffortJointInterface</hardwareInterface>
-      <mechanicalReduction>1</mechanicalReduction>
-    </actuator>
-  </transmission>
-  <transmission name="lb_rot_2_trans">
-    <type>transmission_interface/SimpleTransmission</type>
-    <joint name="lb_rot_2">
-      <hardwareInterface>hardware_interface/EffortJointInterface</hardwareInterface>
-    </joint>
-    <actuator name="lb_rot_2_motor">
-      <hardwareInterface>hardware_interface/EffortJointInterface</hardwareInterface>
-      <mechanicalReduction>1</mechanicalReduction>
-    </actuator>
-  </transmission>
-  <transmission name="lb_rot_3_trans">
-    <type>transmission_interface/SimpleTransmission</type>
-    <joint name="lb_rot_3">
-      <hardwareInterface>hardware_interface/EffortJointInterface</hardwareInterface>
-    </joint>
-    <actuator name="lb_rot_3_motor">
-      <hardwareInterface>hardware_interface/EffortJointInterface</hardwareInterface>
-      <mechanicalReduction>1</mechanicalReduction>
-    </actuator>
-  </transmission>
-  <transmission name="rb_rot_1_trans">
-    <type>transmission_interface/SimpleTransmission</type>
-    <joint name="rb_rot_1">
-      <hardwareInterface>hardware_interface/EffortJointInterface</hardwareInterface>
-    </joint>
-    <actuator name="rb_rot_1_motor">
-      <hardwareInterface>hardware_interface/EffortJointInterface</hardwareInterface>
-      <mechanicalReduction>1</mechanicalReduction>
-    </actuator>
-  </transmission>
-  <transmission name="rb_rot_2_trans">
-    <type>transmission_interface/SimpleTransmission</type>
-    <joint name="rb_rot_2">
-      <hardwareInterface>hardware_interface/EffortJointInterface</hardwareInterface>
-    </joint>
-    <actuator name="rb_rot_2_motor">
-      <hardwareInterface>hardware_interface/EffortJointInterface</hardwareInterface>
-      <mechanicalReduction>1</mechanicalReduction>
-    </actuator>
-  </transmission>
-  <transmission name="rb_rot_3_trans">
-    <type>transmission_interface/SimpleTransmission</type>
-    <joint name="rb_rot_3">
-      <hardwareInterface>hardware_interface/EffortJointInterface</hardwareInterface>
-    </joint>
-    <actuator name="rb_rot_3_motor">
-      <hardwareInterface>hardware_interface/EffortJointInterface</hardwareInterface>
-      <mechanicalReduction>1</mechanicalReduction>
-    </actuator>
-  </transmission>
+  <!-- Transmissions for ros_control -->
+  <xacro:macro name="transmission_block" params="joint_name">
+    <transmission name="trans1">
+      <type>transmission_interface/SimpleTransmission</type>
+      <joint name="${joint_name}">
+        <hardwareInterface>hardware_interface/EffortJointInterface</hardwareInterface>
+      </joint>
+      <actuator name="motor1">
+        <hardwareInterface>hardware_interface/EffortJointInterface</hardwareInterface>
+        <mechanicalReduction>1</mechanicalReduction>
+      </actuator>
+    </transmission>
+  </xacro:macro>
+  <xacro:transmission_block joint_name="lf_rot_1"/>
+  <xacro:transmission_block joint_name="lf_rot_2"/>
+  <xacro:transmission_block joint_name="lf_rot_3"/>
+  <xacro:transmission_block joint_name="rf_rot_1"/>
+  <xacro:transmission_block joint_name="rf_rot_2"/>
+  <xacro:transmission_block joint_name="rf_rot_3"/>
+  <xacro:transmission_block joint_name="lb_rot_1"/>
+  <xacro:transmission_block joint_name="lb_rot_2"/>
+  <xacro:transmission_block joint_name="lb_rot_3"/>
+  <xacro:transmission_block joint_name="rb_rot_1"/>
+  <xacro:transmission_block joint_name="rb_rot_2"/>
+  <xacro:transmission_block joint_name="rb_rot_3"/>
+  <!-- Transmissions for ros_control -->
+  <xacro:macro name="transmission_block2" params="joint_name">
+    <transmission name="trans2">
+      <type>transmission_interface/SimpleTransmission</type>
+      <joint name="${joint_name}">
+        <hardwareInterface>hardware_interface/PositionJointInterface</hardwareInterface>
+      </joint>
+      <actuator name="motor2">
+        <hardwareInterface>hardware_interface/PositionJointInterface</hardwareInterface>
+        <mechanicalReduction>1</mechanicalReduction>
+      </actuator>
+    </transmission>
+  </xacro:macro>
+  <xacro:transmission_block2 joint_name="arm_rot_1"/>
+  <xacro:transmission_block2 joint_name="arm_rot_2"/>
+  <xacro:transmission_block2 joint_name="arm_rot_3"/>
+  <xacro:transmission_block2 joint_name="arm_rot_4"/>
+  <xacro:transmission_block2 joint_name="arm_rot_5"/>
+  <xacro:transmission_block2 joint_name="arm_rot_6"/>
+  <xacro:transmission_block2 joint_name="finger_pri_1"/>
+  <xacro:transmission_block2 joint_name="finger_pri_2"/>
 </robot>
